Commit message: LIDAR included but the xacro files not really used for it. The lidar object has been included as a joint/frame as part of the robot xacro diffbot_description file. This will be improved in later version. Also the real dimention of the lidar is not defined accurately. The defined parameters are just to verify the creation of laser_frame in rviz2.

File: description/urdf/diffbot.urdf.xacro (robot description, xacro)
@@ -8,4 +8,7 @@
   <!-- Import diffbot ros2_control description -->
   <xacro:include filename="$(find diffdrive_arduino)/ros2_control/diffbot.ros2_control.xacro" />
+  <!-- <xacro:include filename="ros2_control.xacro" />
+  <xacro:include filename="lidar.xacro" />
+  <xacro:include filename="camera.xacro" /> -->
   <xacro:diffbot prefix="$(arg prefix)" />
   <xacro:diffbot_ros2_control

File: description/urdf/diffbot_description.urdf.xacro (robot description, xacro)
@@ -157,5 +157,34 @@
           izz="${caster_wheel_mass * 0.4 * (caster_wheel_radius * caster_wheel_radius)}"/>
         </inertial>
-      </link>
+    </link>
+    <joint name="laser_joint" type="fixed">
+      <parent link="${prefix}base_link"/>
+      <child link="laser_frame"/>
+      <origin xyz="0.1 0 0.175" rpy="0 0 0"/>
+    </joint>
+    <!-- LIDAR -->
+    <link name="laser_frame">
+      <collision>
+        <origin xyz="0 0 0" rpy="0 0 0"/>
+        <geometry>
+          <sphere radius="${caster_wheel_radius}"/>
+        </geometry>
+      </collision>
+      <visual>
+        <origin xyz="0 0 0" rpy="0 0 0"/>
+        <geometry>
+          <sphere radius="${caster_wheel_radius}"/>
+        </geometry>
+        <material name="white"/>
+      </visual>
+      <inertial>
+        <origin xyz="0 0 0" rpy="0 0 0"/>
+        <mass value="${caster_wheel_mass}"/>
+        <inertia
+          ixx="${caster_wheel_mass * 0.4 * (caster_wheel_radius * caster_wheel_radius)}" ixy="0.0" ixz="0.0"
+          iyy="${caster_wheel_mass * 0.4 * (caster_wheel_radius * caster_wheel_radius)}" iyz="0.0"
+          izz="${caster_wheel_mass * 0.4 * (caster_wheel_radius * caster_wheel_radius)}"/>
+        </inertial>
+    </link>
   </xacro:macro>
 </robot>
