Commit message: attempted to fix the issue with my_bot description file; still not fixed

File: description/urdf/diffbot_description.urdf.xacro (robot description, xacro)
@@ -14,4 +14,6 @@
   <xacro:property name="caster_wheel_radius" value="0.015" />
   <xacro:property name="z_offset" value="-${base_height/2}" /> <!-- Space btw top of beam and the each joint -->
+  <xacro:property name="lidar_mass" value="0.25" />
+  <xacro:property name="lidar_radius" value="0.025" />
   <!-- Base Link -->
   <link name="${prefix}base_link">
@@ -168,5 +170,5 @@
         <origin xyz="0 0 0" rpy="0 0 0"/>
         <geometry>
-          <sphere radius="${caster_wheel_radius}"/>
+          <sphere radius="${lidar_radius}"/>
         </geometry>
       </collision>
@@ -174,5 +176,5 @@
         <origin xyz="0 0 0" rpy="0 0 0"/>
         <geometry>
-          <sphere radius="${caster_wheel_radius}"/>
+          <sphere radius="${lidar_radius}"/>
         </geometry>
         <material name="white"/>
@@ -180,9 +182,9 @@
       <inertial>
         <origin xyz="0 0 0" rpy="0 0 0"/>
-        <mass value="${caster_wheel_mass}"/>
+        <mass value="${lidar_mass}"/>
         <inertia
-          ixx="${caster_wheel_mass * 0.4 * (caster_wheel_radius * caster_wheel_radius)}" ixy="0.0" ixz="0.0"
-          iyy="${caster_wheel_mass * 0.4 * (caster_wheel_radius * caster_wheel_radius)}" iyz="0.0"
-          izz="${caster_wheel_mass * 0.4 * (caster_wheel_radius * caster_wheel_radius)}"/>
+          ixx="${lidar_mass * 0.4 * (lidar_radius * lidar_radius)}" ixy="0.0" ixz="0.0"
+          iyy="${lidar_mass * 0.4 * (lidar_radius * lidar_radius)}" iyz="0.0"
+          izz="${lidar_mass * 0.4 * (lidar_radius * lidar_radius)}"/>
         </inertial>
     </link>
